File: hardware/eagle/tritiled22.brd (EAGLE design)
At the start: 27.9 x 27.9 mm, 15 parts

Commit message: added names and values to schematic and PCB
Parts:
- C1: value C1206 -> 10u
- C2: value C0805 -> 1u
- D1: value LED_3W -> Chanzon 3W
- L1: value SRR6028_INDUCTOR -> 1m
- Q1: value ZXMN3B01FSOT23 -> ZXMN3B01FTA
- Q2: value DMG2305UXSOT23 -> DMG2305UX
- R1: value R -> 100
- renumbered U$1 to U1, U$12 to D1, U$16 to Q1, U$17 to R1, U$22 to Q2, U$24 to C1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
