File: hardware/eagle/tritiled22_lux_c.sch (EAGLE design)
At the start: 15 parts, among them Q1 ZXMN3B01FTA, Q2 DMG2305UX, SW1 SMD_SWITCH, U1 PIC12LF1571

Commit message: Added new LED eiditons: 5630, Luxeon C, Luxeon Z fixed inconsistent C2 value: now should be 100n everywhere
Parts:
- D1: value Chanzon 3W -> Luxeon C; device tritiled:LED_3W -> tritiled:LEDLUXEON_C
Changed lines of the file:
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@@
 <part name="U$8" library="z0" deviceset="GND" device=""/>
 <part name="U$11" library="z0" deviceset="GND" device=""/>
-<part name="D1" library="tritiled" deviceset="LED_3W" device="" value="Chanzon 3W"/>
+<part name="D1" library="tritiled" deviceset="LED" device="LUXEON_C" value="Luxeon C"/>
 <part name="L1" library="tritiled" deviceset="SRR6028_INDUCTOR" device="" value="1m"/>
 <part name="U$13" library="tritiled" deviceset="+3.0V" device=""/>
