File: hardware/eagle/V3/tritiled_v30_oslon.sch (EAGLE design)
At the start: 12 parts, among them IC1 PIC12LF1571, IC2 74LVC1G123, Q1 IRLML6244, Q2 DMG2305UX

Commit message: updated files for initial V3.0 release
Parts:
- C2: value 100n -> 1u
- D1: value OSLON Signal -> OSLON S.V.
- R3: value 10k -> 51k
- renumbered U$1 to D1
Changed lines of the file:
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@@
 <?xml version="1.0" encoding="utf-8"?>
 <!DOCTYPE eagle SYSTEM "eagle.dtd">
-<eagle version="8.2.2">
+<eagle version="8.5.0">
 <drawing>
 <settings>
 <setting alwaysvectorfont="yes"/>
+<setting keepoldvectorfont="yes"/>
 <setting verticaltext="up"/>
 </settings>
@@
 <layers>
 <layer number="1" name="Top" color="4" fill="1" visible="no" active="no"/>
+<layer number="2" name="Route2" color="1" fill="3" visible="no" active="no"/>
+<layer number="15" name="Route15" color="4" fill="6" visible="no" active="no"/>
 <layer number="16" name="Bottom" color="1" fill="1" visible="no" active="no"/>
 <layer number="17" name="Pads" color="2" fill="1" visible="no" active="no"/>
@@
 </classes>
 <parts>
-<part name="U$1" library="tritiled" deviceset="OSLON_SIGNAL" device="" value="OSLON Signal"/>
+<part name="D1" library="tritiled" deviceset="OSLON_SIGNAL" device="" value="OSLON S.V."/>
 <part name="B1" library="tritiled" deviceset="BAT-HLD-001-THM_CR2032" device=""/>
 <part name="U$3" library="tritiled" deviceset="GND" device=""/>
@@
 <part name="U$13" library="tritiled" deviceset="GND" device=""/>
 <part name="U$14" library="tritiled" deviceset="+3.0V" device=""/>
-<part name="C2" library="tritiled" deviceset="C" device="0805" value="100n"/>
+<part name="C2" library="tritiled" deviceset="C" device="0805" value="1u"/>
 <part name="U$15" library="tritiled" deviceset="GND" device=""/>
 <part name="U$16" library="tritiled" deviceset="+3.0V" device=""/>
@@
 <part name="IC2" library="tritiled" deviceset="74LVC1G123" device=""/>
 <part name="U$22" library="tritiled" deviceset="GND" device=""/>
-<part name="R3" library="tritiled" deviceset="R" device="0603" value="10k"/>
+<part name="R3" library="tritiled" deviceset="R" device="0603" value="51k"/>
 <part name="C5" library="tritiled" deviceset="C" device="0603" value="100p"/>
 <part name="Q2" library="tritiled" deviceset="DMG2305UX" device="SOT23" value="DMG2305UX"/>
@@
 </plain>
 <instances>
-<instance part="U$1" gate="G$1" x="76.2" y="63.5" rot="MR180"/>
+<instance part="D1" gate="G$1" x="76.2" y="63.5" rot="MR180"/>
 <instance part="B1" gate="G$1" x="-193.04" y="33.02"/>
 <instance part="U$3" gate="G$1" x="-193.04" y="20.32"/>
@@
 <pinref part="L1" gate="G$1" pin="1"/>
 <wire x1="55.88" y1="86.36" x2="55.88" y2="78.74" width="0.1524" layer="91"/>
-<pinref part="U$1" gate="G$1" pin="C"/>
+<pinref part="D1" gate="G$1" pin="C"/>
 <wire x1="55.88" y1="78.74" x2="55.88" y2="71.12" width="0.1524" layer="91"/>
 <wire x1="76.2" y1="71.12" x2="76.2" y2="78.74" width="0.1524" layer="91"/>
@@
 <pinref part="L1" gate="G$1" pin="2"/>
 <pinref part="Q1" gate="G$1" pin="D"/>
-<pinref part="U$1" gate="G$1" pin="A"/>
+<pinref part="D1" gate="G$1" pin="A"/>
 <wire x1="76.2" y1="55.88" x2="76.2" y2="50.8" width="0.1524" layer="91"/>
 <wire x1="76.2" y1="50.8" x2="55.88" y2="50.8" width="0.1524" layer="91"/>
