File: hardware/eagle/V3/tritiled_v30_lux_c.brd (EAGLE design)
At the start: 22.9 x 22.9 mm, 12 parts, among them IC1 PIC12LF1571, IC2 74LVC1G123, Q1 IRLML6244, Q2 DMG2305UX

Commit message: correct values for R3
Parts:
- R3: value 10k -> 75k
Changed lines of the file:
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@@
 <?xml version="1.0" encoding="utf-8"?>
 <!DOCTYPE eagle SYSTEM "eagle.dtd">
-<eagle version="8.2.2">
+<eagle version="8.5.0">
 <drawing>
 <settings>
 <setting alwaysvectorfont="yes"/>
+<setting keepoldvectorfont="yes"/>
 <setting verticaltext="up"/>
 </settings>
@@
 <param name="dpMaxLengthDifference" value="10mm"/>
 <param name="dpGapFactor" value="2.5"/>
-<param name="checkGrid" value="0"/>
 <param name="checkAngle" value="1"/>
 <param name="checkFont" value="1"/>
 <param name="checkRestrict" value="1"/>
+<param name="checkStop" value="0"/>
+<param name="checkValues" value="0"/>
 <param name="useDiameter" value="13"/>
 <param name="maxErrors" value="50"/>
@@
 <element name="C3" library="tritiled" package="1206" value="10u" x="11.43" y="15.875"/>
 <element name="IC2" library="tritiled" package="SM8" value="74LVC1G123" x="11.43" y="3.81" rot="R90"/>
-<element name="R3" library="tritiled" package="R0603" value="10k" x="6.35" y="3.81" rot="R180"/>
+<element name="R3" library="tritiled" package="R0603" value="75k" x="6.35" y="3.81" rot="R180"/>
 <element name="C5" library="tritiled" package="C0603" value="100p" x="6.35" y="6.0325" rot="R180"/>
 <element name="Q2" library="tritiled" package="SOT-23" value="DMG2305UX" x="16.1925" y="6.0325" rot="R90"/>
